Commit message: torque control

File: src/factr_teleop/factr_teleop/urdf/factr_teleop_franka.urdf (robot description, URDF)
Before this commit: robot factr_teleop_franka, 8 links, 7 joints
Links:
- link link_3: mass 0.113 -> 0.103
- link link_4: mass 0.051 -> 0.041
- link link_5: mass 0.048 -> 0.038
